File: Conexión entre 2 arduinos/Conexión entre 2 arduinos.brd (EAGLE design)
At the start: 138.8 x 84 mm, 2 parts, among them U1 ARDUINO-UNO-R3-SHIELD, U2 ARDUINO-UNO-R3-SHIELD

Commit message: Se corrigen errores. Se envía una trama de informacion del arduino uno al dos, se recibe adecuadamente. Hay sincronismo
Connections:
- new net U1_D13: U1.D13, U2.D13
Changed lines of the file:
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@@
 <wire x1="133.0601" y1="50.425" x2="133.0601" y2="52.965" width="0" layer="19" extent="1-1"/>
+</signal>
+<signal name="U1_D13">
+<contactref element="U1" pad="D13"/>
+<contactref element="U2" pad="D13"/>
+<wire x1="53.975" y1="44.9695" x2="84.8001" y2="38.995" width="0" layer="19" extent="1-1"/>
 </signal>
 <signal name="U1_D6">
